Commit message: updated right urdf values, reference left

File: src/ah_urdf/urdf/ability_hand_right_large.urdf (robot description, URDF)
Before this commit: robot ability_hand, 47 links, 46 joints
Links:
- link pinky_L2: geometry collision mesh filename=package://ah_urdf/models/idx-F2-hull.STL; visual mesh filename=package://ah_urdf/models/idx-F2-Lg.STL
Joints:
- joint fsr24: origin xyz=0.04747 0.01988 -0.001239 rpy=-2.29074 0.00001 0.41769 -> xyz=0.04747 0.01988 0.00874 rpy=-2.29074 0.00001 0.41769
- joint fsr25: origin xyz=0.04721 0.02124 0.006439 rpy=-1.30899 0.00001 0.41769 -> xyz=0.04721 0.02124 0.00106 rpy=-1.30899 0.00001 0.41769
- joint fsr26: origin xyz=0.04896 0.01654 0.01241 rpy=-0.32726 0.00001 0.41769 -> xyz=0.04896 0.01654 -0.00491 rpy=-0.32726 0.00001 0.41769
- joint fsr27: origin xyz=0.03739 0.01536 -0.001289 rpy=-2.29074 0.00001 0.41769 -> xyz=0.03739 0.01536 +0.00879 rpy=-2.29074 0.00001 0.41769
- joint fsr28: origin xyz=0.03888 0.01200 0.01244 rpy=-0.32726 0.00001 0.41769 -> xyz=0.03888 0.01200 -0.00494 rpy=-0.32726 0.00001 0.41769
- joint fsr29: origin xyz=0.05591 0.02160 0.00558 rpy=-1.39339 0.19354 -0.40280 -> xyz=0.05591 0.02160 0.00192 rpy=-1.39339 0.19354 -0.40280
- joint thmb_anchor: origin xyz=52.00122724e-3 28.00869333e-3 6.98483578e-3 rpy=0 0 0 -> xyz=52.00122724e-3 28.00869333e-3 0.884835778e-3 rpy=0 0 0
